Commit message: make simviz_Gordon_robot work

File: Gordon_the_robot/urdf_files/mmp_panda.urdf (robot description, URDF)
Before this commit: robot mmp_panda, 13 links, 12 joints
Links:
- link base_link: geometry visual mesh filename=../../../Gordon_the_robot/model/mmp_panda/meshes/panda_Base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
- link leftfinger: geometry collision mesh filename=../../../Gordon_the_robot/model/panda/meshes/collision/fing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 scale=5.0 1.0 2.5; visual mesh filename=../../../Gordon_the_robot/model/panda/meshes/collision/fing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 scale=5.0 1.0 2.5
- link link1: geometry visual mesh filename=../../../Gordon_the_robot/model/panda/meshes/visual/link1.o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
- link link2: geometry visual mesh filename=../../../Gordon_the_robot/model/panda/meshes/visual/link2.o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
- link link3: geometry visual mesh filename=../../../Gordon_the_robot/model/panda/meshes/visual/link3.o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
- link link4: geometry visual mesh filename=../../../Gordon_the_robot/model/panda/meshes/visual/link4.o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
- link link5: geometry visual mesh filename=../../../Gordon_the_robot/model/panda/meshes/visual/link5.o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
- link link6: geometry visual mesh filename=../../../Gordon_the_robot/model/panda/meshes/visual/link6.o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
- link link7: geometry collision mesh filename=../../../Gordon_the_robot/model/panda/meshes/collision/hand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; visual mesh filename=../../../Gordon_the_robot/model/panda/meshes/visual/chefhat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 scale=0.01 0.01 0.01
- link rightfinger: geometry collision mesh filename=../../../Gordon_the_robot/model/panda/meshes/collision/fing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 scale=5.0 1.0 1.5; visual mesh filename=../../../Gordon_the_robot/model/panda/meshes/collision/fing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 scale=5.0 1.0 1.5
